File: mbus.kicad_pcb (KiCad board)
At the start: 2 copper layers, 62.9 x 27.2 mm, 37 parts, among them J1 USB_C_Receptacle_USB2.0, J2 MBUS, Q1 BC817, Q2 BC817, Q3 BC807, U1 AP3015, U2 USBLC6-2SC6, U3 CH340E

Commit message: rev 0.2 - swapped RX/TX pins
Parts:
- added NT1: NetTie_2, NetTie:NetTie-2_SMD_Pad0.5mm, F.Cu at (90.8, 75.0)
- added kibuzzard-62A19C5B: G***, kibuzzard-62A19C5B, F.Cu at (92.6, 90.8)
- C4, C5, C6: footprint Capacitor_SMD:C_0402_1005Metric -> Capacitor_SMD:C_0603_1608Metric
- D3: value 5.0SMDJ36A -> SMBJ36A; footprint Diode_SMD:D_SMC -> Diode_SMD:D_SMB
- R1, R2: footprint Resistor_SMD:R_0402_1005Metric -> Resistor_SMD:R_0603_1608Metric
- R3: value 1.8M -> 1.02M
- R4: value 68k -> 39k
- moved G*** 3.58 mm to (91.6, 87.2)
- moved H2 3.38 mm to (100.4, 69.0)
- moved H3 3.38 mm to (100.4, 91.2)
- moved J2 2.55 mm to (98.1, 81.1)
- moved D3 1.30 mm to (90.8, 78.5)
- moved C4 1.21 mm to (60.0, 80.4), turned to 180 degrees
- moved C5 0.92 mm to (63.2, 80.4), turned to 0 degrees
- moved C6 0.85 mm to (65.7, 74.9)
- moved R2 0.71 mm to (53.0, 73.2)
- moved R1 0.67 mm to (53.0, 79.8)
Connections:
- J1 pad S1: (no net) -> unconnected-(J1-PadS1)
- R5 pad 1: /UART_TX -> /UART_RX
- R6 pad 1: /UART_RX -> /UART_TX
Routing:
- net /UART_TX: track 14.0 -> 2.23 mm
- net /UART_RX: track 2.44 -> 8.61 mm
- net /-: track 22.3 -> 19.0 mm
- net /+: track 19.7 -> 16.4 mm
- net GND: track 8.80 -> 10.8 mm, vias 21 -> 22
- net VBUS: track 29.6 -> 31.0 mm
- net +34V: track 29.0 -> 28.5 mm, vias 2 -> 0
Other:
- board size 62.9 x 27.2 mm -> 59.5 x 27.2 mm
- board text added: "7/22"
- board text added: "Designed by"
- board text added: "rev0.2"
- board text removed: "4/22"
- board text removed: "Designed by Jan Gnip"
- board text removed: "rev0.1"
